File: Schematic_kicad/schematic kicad.kicad_sch (KiCad schematic)
At the start: 18 parts

Commit message: minor fixes
Connections:
- net +5V: now also U?.1 (~{RST})
- net ESP_TX: now reaches U?.16 (TX)
Other:
- note added: "I used the Arduino MEGA board, therefore, the labels in the MCU refer to the board's pins: PIN[FUNCTION]. If FUNCTION is not specified, it is the default one. Also note that the RESET is pulled up inside of the board. The pins that are not connected to anything nor marked as unconnected are the ones that are not mapped to any pin on the Arduino board (but connected internally)"
- note added: "This capacitor is not necessary, the Arduino boards reset when the serial connection is established. It is a feature, they did it to enter the bootloader during the MCU programming, but it can cause problems in applications like this. In the board there is the possibility to cut the little link to stop it from doing that. Indead of cutting the link, this capacitor can prevent the board from reset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"
- note removed: "I used the Arduino MEGA board, therefore the labels in the MCU refer to the board's pins: PIN[FUNCTION]. If FUNCTION is not specified, it is the default one. Also note that the RESET is pulled up inside of the board."
- note removed: "This capacitor is not necessary if you are not using the Arduino board. The Arduino boards reset when the serial connection is established. It is a feature, they did it to enter the bootloader during the MCU programming, but it can cause problems in applications like this. In the board there is the possibility to cut the little link to stop it from doing that. Indead of cutting the link, this cap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"
- moved on the sheet: 10k, 56ohm
